Commit message: sim world is up, can run but without imu yet.

File: src/dream_base_description/urdf/diff_drive.gazebo.xacro (robot description, xacro)
@@ -1,44 +1,15 @@
 <?xml version="1.0"?>
-<robot name="nuturtle_gazebo" xmlns:xacro="http://www.ros.org/wiki/xacro">
+<robot name="dream_gazebo_diff_drive" xmlns:xacro="http://www.ros.org/wiki/xacro">
     <!-- Notes: load urdf, then load diff params -->
-    <xacro:include filename="$(find nuturtle_description)/urdf/diff_drive.urdf.xacro" />
-    <xacro:property name="diff_params" value="${load_yaml('$(find nuturtle_description)/config/diff_params.yaml')}" />
-    <!--    specify link properties like this?-->
-    <!-- diffdrive source code: https://github.com/ros-simulation/gazebo_ros_pkgs/blob/noetic-devel/gazebo_plugins/src/gazebo_ros_diff_drive.cpp  -->
+    <xacro:include filename="$(find dream_base_description)/urdf/diff_drive.urdf.xacro" />
+    <xacro:property name="diff_params" value="${load_yaml('$(find dream_base_description)/config/diff_params.yaml')}" />`
     <gazebo>
-        <plugin name="differential_drive_controller" filename="libgazebo_ros_diff_drive.so">
-        <legacyMode>false</legacyMode>
-        <alwaysOn>true</alwaysOn>
-        <updateRate>10</updateRate>
-        <leftJoint>left_wheel_hinge</leftJoint>
-        <rightJoint>right_wheel_hinge</rightJoint>
-        <wheelSeparation>0.4</wheelSeparation>
-        <wheelDiameter>0.2</wheelDiameter>
-        <torque>10</torque>
-        <commandTopic>cmd_vel</commandTopic>
-        <odometryTopic>odom</odometryTopic>
-        <odometryFrame>odom</odometryFrame>
-        <robotBaseFrame>robot_footprint</robotBaseFrame>
-        <publishWheelTF>false</publishWheelTF>
-        <publishWheelJointState>false</publishWheelJointState>
-        <rosDebugLevel>na</rosDebugLevel>
-        <wheelAcceleration>0</wheelAcceleration>
-        <wheelTorque>5</wheelTorque>
-        <odometrySource>world</odometrySource>
-        <publishTf>1</publishTf>
-        <publishOdomTF>true</publishOdomTF>
-        </plugin>
-    </gazebo>
-    <gazebo>
-        <!-- <plugin name="turtle_drive_plugin" filename="libnuturtle_gazebo_plugin.so">
+        <!-- Notes: use params loaded from yaml -->
+        <plugin name="dream_gazebo_diff_drive_plugin" filename="libdream_gazebo_diff_drive_plugin.so">
             <left_wheel_joint>left_wheel_axle</left_wheel_joint>
             <right_wheel_joint>right_wheel_axle</right_wheel_joint>
-            <sensor_frequency> 60 </sensor_frequency>
-            <wheel_cmd_topic>wheel_cmd</wheel_cmd_topic>
-            <sensor_data_topic>sensor_data</sensor_data_topic>
-            <max_wheel_command>${diff_params['max_wheel_command']}</max_wheel_command>
-            <max_motor_rot_vel>${diff_params['max_motor_rot_vel']}</max_motor_rot_vel>
-            <encoder_ticks_per_rev>${diff_params['encoder_ticks_per_rev']}</encoder_ticks_per_rev>
-        </plugin> -->
+            <wheel_radius>${diff_params['wheel_radius']}</wheel_radius>
+            <commanded_wheel_vel_topic>${diff_params['commanded_wheel_vel_topic']}</commanded_wheel_vel_topic>
+        </plugin>
     </gazebo>
     <gazebo reference="base_link">

File: src/dream_base_description/urdf/diff_drive.urdf.xacro (robot description, xacro)
@@ -1,5 +1,5 @@
 <?xml version="1.0"?>
 <robot xmlns:xacro="http://www.ros.org/wiki/xacro" name="diff_drive">
-    <xacro:property name="diff_params" value="${load_yaml('$(find nuturtle_description)/config/diff_params.yaml')}" />
+    <xacro:property name="diff_params" value="${load_yaml('$(find dream_base_description)/config/diff_params.yaml')}" />
     <xacro:property name="grey_mat">
      <material name="arm_grey_mat">
@@ -166,5 +166,5 @@
     </link>
     <xacro:_joint name="left_wheel_axle"
-           type="fixed"
+           type="continuous"
            origin_xyz = "0.0 ${0.5*diff_params['wheel_base']} ${diff_params['wheel_axle_offset']}" origin_rpy="0 0 0"
            parent = "chassis"
@@ -177,5 +177,5 @@
              radius="${diff_params['wheel_radius']}"/>
     <xacro:_joint name="right_wheel_axle"
-        type="fixed"
+        type="continuous"
         origin_xyz = "0.0 ${-0.5*diff_params['wheel_base']} ${diff_params['wheel_axle_offset']}" origin_rpy="0 0 0"
         parent = "chassis"
@@ -208,8 +208,8 @@
           </collision>
           <inertial>
-              <mass value="${100 * diff_params['wheel_mass']}" />
-              <inertia ixx="${diff_params['chassis_mass']*((diff_params['wheel_base']-diff_params['wheel_width'])*(diff_params['wheel_base']-diff_params['wheel_width'])+diff_params['chassis_thickness']*diff_params['chassis_thickness'])/12}" ixy="0.0" ixz="0.0"
-                       iyy="${diff_params['chassis_mass']*(diff_params['chassis_length']*diff_params['chassis_length']+diff_params['chassis_thickness']*diff_params['chassis_thickness'])/12}" iyz="0.0"
-                       izz="${diff_params['chassis_mass']*((diff_params['wheel_base']-diff_params['wheel_width'])*(diff_params['wheel_base']-diff_params['wheel_width'])+diff_params['chassis_length']*diff_params['chassis_length'])/2}" />
+              <mass value="${100 * diff_params['caster_mass']}" />
+              <inertia ixx="${diff_params['caster_mass']*((diff_params['wheel_base']-diff_params['wheel_width'])*(diff_params['wheel_base']-diff_params['wheel_width'])+diff_params['chassis_thickness']*diff_params['chassis_thickness'])/12}" ixy="0.0" ixz="0.0"
+                       iyy="${diff_params['caster_mass']*(diff_params['chassis_length']*diff_params['chassis_length']+diff_params['chassis_thickness']*diff_params['chassis_thickness'])/12}" iyz="0.0"
+                       izz="${diff_params['caster_mass']*((diff_params['wheel_base']-diff_params['wheel_width'])*(diff_params['wheel_base']-diff_params['wheel_width'])+diff_params['chassis_length']*diff_params['chassis_length'])/2}" />
           </inertial>
       </link>

Commit message: rviz

File: src/dream_base_description/urdf/diff_drive.gazebo.xacro (robot description, xacro)
@@ -99,3 +99,42 @@
         </sensor>
     </gazebo>
+    <!-- in URDF, camera will face along the x axis of rgbd_camera -->
+    <gazebo reference="rgbd_camera">
+        <sensor type="depth" name="camera_sensor">
+            <update_rate>10</update_rate> <!-- Frame rate -->
+            <camera>
+                <horizontal_fov>1.047</horizontal_fov> <!-- Field of View -->
+                <image>
+                    <width>640</width>
+                    <height>480</height>
+                    <format>R8G8B8</format>
+                </image>
+                <clip>
+                    <near>0.1</near>
+                    <far>10</far>
+                </clip>
+                <depth>
+                    <near>0.1</near>
+                    <far>10</far>
+                </depth>
+            </camera>
+            <plugin name="camera_plugin" filename="libgazebo_ros_openni_kinect.so">
+                <baseline>0.2</baseline>
+                <alwaysOn>true</alwaysOn>
+                <!-- Keep this zero, update_rate in the parent <sensor> tag
+                will control the frame rate. -->
+                <updateRate>0.0</updateRate>
+                <cameraName>camera_ir</cameraName>
+                <imageTopicName>/camera/color/image_raw</imageTopicName>
+                <cameraInfoTopicName>/camera/color/camera_info</cameraInfoTopicName>
+                <depthImageTopicName>/camera/depth/image_raw</depthImageTopicName>
+                <depthImageCameraInfoTopicName>/camera/depth/camera_info</depthImageCameraInfoTopicName>
+                <pointCloudTopicName>/camera/depth/points</pointCloudTopicName>
+                <!-- This is the frame in which gazebo projects onto -->
+                <frameName>rgbd_camera_projection</frameName>
+                <pointCloudCutoff>0.05</pointCloudCutoff>
+                <pointCloudCutoffMax>10</pointCloudCutoffMax>
+            </plugin>
+        </sensor>
+    </gazebo>
 </robot>

File: src/dream_base_description/urdf/diff_drive.urdf.xacro (robot description, xacro)
@@ -138,4 +138,27 @@
         </inertial>
     </link>
+    <!-- Dummy rgbd camera link that's 30cm above the base link-->
+    <xacro:_joint name="base_link_rgbd_camera"
+                type="fixed"
+                origin_xyz ="0 0  0.3" origin_rpy="0 0 0"
+                parent = "base_link"
+                child = "rgbd_camera"
+                axis = "1 0 0"/>
+    <link name="rgbd_camera">
+        <visual>
+            <origin xyz="0 0 0" rpy="0 0 0"/>
+            <geometry>
+                <box size="0.0001 0.0001 0.0001"/>
+            </geometry>
+            <xacro:insert_block name="pink_mat"/>
+        </visual>
+    </link>
+    <xacro:_joint name="rgbd_camera_rgbd_camera_projection"
+                type="fixed"
+                origin_xyz ="0 0  0.0" origin_rpy="-1.57079 0 -1.57079"
+                parent = "rgbd_camera"
+                child = "rgbd_camera_projection"
+                axis = "1 0 0"/>
+    <link name="rgbd_camera_projection"></link>
     <xacro:_joint name="base_link_chassis"
                   type="fixed"
